File: Pcb/OpenDrift Pdb/OpenDrift Pdb.kicad_pcb (KiCad board)
At the start: 4 copper layers, 29.1 x 44 mm, 12 parts, among them J1 Servo_In, J2 Esc_In, J3 Servo_Out, J4 Esc_out, J5 Conn_01x11_Pin, J6 Conn_01x11_Pin, U2 TPS62162DSG

Commit message: Release OpenDrift v1.0.7 anti-wobble control
Connections:
- U2 pad 3: unconnected-(U2-EN-Pad3) -> +5V
- U2 pad 5: unconnected-(U2-FB-Pad5) -> GND
Routing:
- net GND: track 13.6 -> 14.9 mm
- net +5V: track 75.3 -> 75.8 mm
