File: Pcb/OpenDrift Pdb/OpenDrift Pdb.kicad_sch (KiCad schematic)
At the start: 12 parts, among them J1 Servo_In, J2 Esc_In, J3 Servo_Out, J4 Esc_out, J5 Conn_01x11_Pin, J6 Conn_01x11_Pin, U2 TPS62162DSG

Commit message: Release OpenDrift v1.0.7 anti-wobble control
Connections:
- net +5V: now also U2.3 (EN)
- net GND: now also U2.5 (FB)
Changed lines of the file:
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@@
 	(paper "A4")
 	(junction
+		(at 140.97 31.75)
+		(diameter 0)
+		(color 0 0 0 0)
+	)
+	(junction
 		(at 151.13 59.69)
 		(diameter 0)
@@
 	)
 	(junction
+		(at 161.29 59.69)
+		(diameter 0)
+		(color 0 0 0 0)
+	)
+	(junction
 		(at 80.01 31.75)
 		(diameter 0)
@@
 	(wire
 		(pts
-			(xy 153.67 59.69) (xy 162.56 59.69)
+			(xy 153.67 59.69) (xy 161.29 59.69)
 		)
 		(stroke
@@
 	(wire
 		(pts
+			(xy 140.97 31.75) (xy 140.97 34.29)
+		)
+		(stroke
+			(width 0)
+			(type default)
+		)
+	)
+	(wire
+		(pts
 			(xy 186.69 40.64) (xy 186.69 59.69)
 		)
@@
 	(wire
 		(pts
+			(xy 161.29 36.83) (xy 161.29 59.69)
+		)
+		(stroke
+			(width 0)
+			(type default)
+		)
+	)
+	(wire
+		(pts
 			(xy 186.69 31.75) (xy 186.69 35.56)
 		)
@@
 		)
 		(stroke
+			(width 0)
+			(type default)
+		)
+	)
+	(wire
+		(pts
+			(xy 161.29 59.69) (xy 162.56 59.69)
+		)
+		(stroke
